Commit message: Camera/gravity now fixed

File: urdf/simulated_camera.gazebo.xacro (robot description, xacro)
@@ -49,9 +49,9 @@
 	</link>
 	<joint name="optical_joint" type="fixed">
-		<origin xyz="0 0 0" rpy="0 0 0"/>
+		<origin xyz="0 0 0" rpy="0 ${M_PI/2} 0"/>
 		<parent link="body_link"/>
-		<child link="optical_frame"/>
+		<child link="optical_link"/>
 	</joint>
-	<link name="optical_frame">
+	<link name="optical_link">
 		<inertial>
 			<mass value="1" />
@@ -69,13 +69,13 @@
 		<gravity>0</gravity>
 	</gazebo>
-<!-- 	<gazebo reference="optical_frame">
+	<gazebo reference="optical_link">
 		<gravity>0</gravity>
-	</gazebo> -->
-<!-- 	<gazebo reference="base_link">
+	</gazebo>
+	<gazebo reference="optical_link">
 		<gravity>0</gravity>
 		<sensor type="camera" name="$(arg name)_camera_sensor">
 			<update_rate>$(arg update_rate)</update_rate>
 			<camera>
-				<horizontal_fov>$(arg hfov) * M_PI/180.0</horizontal_fov>
+				<horizontal_fov>${$(arg hfov) * M_PI/180.0}</horizontal_fov>
 				<image>
 					<format>$(arg image_format)</format>
@@ -92,7 +92,7 @@
 				<imageTopicName>$(arg ros_topic)</imageTopicName>
 				<cameraInfoTopicName>$(arg cam_info_topic)</cameraInfoTopicName>
-				<frameName>optical_frame</frameName>
+				<frameName>optical_link</frameName>
 			</plugin>
 		</sensor>
-	</gazebo> -->
+	</gazebo>
 </robot>

Commit message: Grid simulator with camera now fully finished!

File: urdf/simulated_camera.gazebo.xacro (robot description, xacro)
@@ -49,5 +49,5 @@
 	</link>
 	<joint name="optical_joint" type="fixed">
-		<origin xyz="0 0 0" rpy="0 ${M_PI/2} 0"/>
+		<origin xyz="0 0 -0.15" rpy="0 ${M_PI/2} 0"/>
 		<parent link="body_link"/>
 		<child link="optical_link"/>
